File: pcb/driver-board/driver-board.kicad_sch (KiCad schematic)
At the start: 116 parts, among them Q1 IRLML6344, Q10 IRLML6344, Q11 IRLML6344, Q12 2N7002, Q2 IRLML6344, Q3 IRLML6344, Q4 IRLML6344, Q5 IRLML6344, Q6 IRLML6344, Q7 IRLML6344, Q8 IRLML6344, Q9 IRLML6344, U1 MP1584EN_12V, U2 MP1584EN_6V5, U3 MP1584EN_5V, U4 DRV8876, U5 DRV8876, U6 TB6612FNG, U7 INA219, U8 PCF8574

Commit message: Add files via upload
Finalize schematics: 0 ERC errors, subsystem boxes added
Parts:
- removed C_BULK1: 470uF/10V, Capacitor_THT:CP_Radial_D8.0mm_P3.50mm, symbol Device:C_Polarized
- removed C_BULK3: 100uF/25V, Capacitor_THT:CP_Radial_D6.3mm_P2.50mm, symbol Device:C_Polarized
- removed C_BULK5V: 220uF/10V, Capacitor_THT:CP_Radial_D6.3mm_P2.50mm, symbol Device:C_Polarized
- removed C_IN1, C_IN2, C_IN3: 10uF, Capacitor_SMD:C_0805_2012Metric, symbol Device:C
- removed C_OUT1a, C_OUT1b, C_OUT2a, C_OUT2b, C_OUT3a, C_OUT3b: 22uF, Capacitor_SMD:C_0805_2012Metric, symbol Device:C
- removed C_VCC6, C_VDD8, C_VM4, C_VM5, C_VM6, C_VS7: 100nF, Capacitor_SMD:C_0402_1005Metric, symbol Device:C
- removed D1: SS54, Diode_SMD:D_SMA, symbol Diode:SS54
- removed D10, D11, D12, D13, D14, D15, D16, D6, D7, D8, D9: SS14, Diode_SMD:D_SMA, symbol Diode:SS54
- removed D2: SMBJ24A, Diode_SMD:D_SMB, symbol Device:C
- removed D3: SMBJ12A, Diode_SMD:D_SMB, symbol Device:C
- removed D4: SMBJ6.5A, Diode_SMD:D_SMB, symbol Device:C
- removed D5: SMBJ5.0A, Diode_SMD:D_SMB, symbol Device:C
- removed D_BST1, D_BST2, D_BST3: SS34, Diode_SMD:D_SMA, symbol Diode:SS54
- removed F1: 5A, Resistor_SMD:R_1812_4532Metric, symbol Device:Polyfuse
- removed F2: 1.5A, Resistor_SMD:R_0805_2012Metric, symbol Device:Polyfuse
- removed F3: 3A, Resistor_SMD:R_1206_3216Metric, symbol Device:Polyfuse
- removed F4: 2A, Resistor_SMD:R_1206_3216Metric, symbol Device:Polyfuse
- removed J_24V_IN: XT30, Connector_XT:XT30PW-M, symbol Connector_Generic:Conn_01x02
- removed J_BUZZER: Buzzer, Connector_JST:JST_PH_B2B-PH-K_1x02_P2.00mm_Vertical, symbol Connector_Generic:Conn_01x02
- removed J_CID_LACT1: CID_LACT1, Connector_JST:JST_XH_B2B-XH-A_1x02_P2.50mm_Vertical, symbol Connector_Generic:Conn_01x02
- removed J_CID_LACT2: CID_LACT2, Connector_JST:JST_XH_B2B-XH-A_1x02_P2.50mm_Vertical, symbol Connector_Generic:Conn_01x02
- removed J_FAN1: Fan1, Connector_JST:JST_XH_B2B-XH-A_1x02_P2.50mm_Vertical, symbol Connector_Generic:Conn_01x02
- removed J_FAN2: Fan2, Connector_JST:JST_XH_B2B-XH-A_1x02_P2.50mm_Vertical, symbol Connector_Generic:Conn_01x02
- removed J_MAIN_SERVO: DS3225, Connector_PinHeader_2.54mm:PinHeader_1x03_P2.54mm_Vertical, symbol Connector_Generic:Conn_01x03
- removed J_PASD_PUMP: PASD_Pump, Connector_JST:JST_XH_B2B-XH-A_1x02_P2.50mm_Vertical, symbol Connector_Generic:Conn_01x02
- removed J_PASD_SOL1: PASD_SOL1, Connector_JST:JST_XH_B2B-XH-A_1x02_P2.50mm_Vertical, symbol Connector_Generic:Conn_01x02
- removed J_PASD_SOL2: PASD_SOL2, Connector_JST:JST_XH_B2B-XH-A_1x02_P2.50mm_Vertical, symbol Connector_Generic:Conn_01x02
- removed J_PASD_SOL3: PASD_SOL3, Connector_JST:JST_XH_B2B-XH-A_1x02_P2.50mm_Vertical, symbol Connector_Generic:Conn_01x02
- removed J_PASD_SOL4: PASD_SOL4, Connector_JST:JST_XH_B2B-XH-A_1x02_P2.50mm_Vertical, symbol Connector_Generic:Conn_01x02
- removed J_PASD_SOL5: PASD_SOL5, Connector_JST:JST_XH_B2B-XH-A_1x02_P2.50mm_Vertical, symbol Connector_Generic:Conn_01x02
- removed J_PASD_SOL6: PASD_SOL6, Connector_JST:JST_XH_B2B-XH-A_1x02_P2.50mm_Vertical, symbol Connector_Generic:Conn_01x02
- removed J_SLD: SLD, Connector_JST:JST_XH_B8B-XH-A_1x08_P2.50mm_Vertical, symbol Connector_Generic:Conn_01x08
- removed J_SLD_SOL1: SLD_SOL1, Connector_JST:JST_XH_B2B-XH-A_1x02_P2.50mm_Vertical, symbol Connector_Generic:Conn_01x02
- removed J_SLD_SOL2: SLD_SOL2, Connector_JST:JST_XH_B2B-XH-A_1x02_P2.50mm_Vertical, symbol Connector_Generic:Conn_01x02
- removed J_STACK: J_STACK, Connector_PinSocket_2.54mm:PinSocket_2x20_P2.54mm_Vertical, symbol Connector_Generic:Conn_02x20_Odd_Even
- removed L1: 33uH, Inductor_SMD:L_1210_3225Metric, symbol Device:L
- removed L2, L3: 22uH, Inductor_SMD:L_1210_3225Metric, symbol Device:L
- removed Q1, Q10, Q11, Q2, Q3, Q4, Q5, Q6, Q7, Q8, Q9: IRLML6344, Package_TO_SOT_SMD:SOT-23, symbol Transistor_FET:IRLML6344
- removed R_FB1_BOT, R_FB2_BOT, R_FB3_BOT, R_Q10_PD, R_Q11_PD, R_Q12_PD, R_Q1_PD, R_Q2_PD, R_Q3_PD, R_Q4_PD, R_Q5_PD, R_Q6_PD, R_Q7_PD, R_Q8_PD, R_Q9_PD: 10k, Resistor_SMD:R_0402_1005Metric, symbol Device:R
- removed R_FB1_TOP: 140k, Resistor_SMD:R_0402_1005Metric, symbol Device:R
- removed R_FB2_TOP: 71.5k, Resistor_SMD:R_0402_1005Metric, symbol Device:R
- removed R_FB3_TOP: 52.3k, Resistor_SMD:R_0402_1005Metric, symbol Device:R
- removed R_Q10_GATE, R_Q11_GATE, R_Q12_GATE, R_Q1_GATE, R_Q2_GATE, R_Q3_GATE, R_Q4_GATE, R_Q5_GATE, R_Q6_GATE, R_Q7_GATE, R_Q8_GATE, R_Q9_GATE: 100R, Resistor_SMD:R_0402_1005Metric, symbol Device:R
- removed R_SENSE1, R_SENSE2: 1k, Resistor_SMD:R_0402_1005Metric, symbol Device:R
- removed R_SERVO: 33R, Resistor_SMD:R_0402_1005Metric, symbol Device:R
- removed R_SHUNT: 10mR, Resistor_SMD:R_2512_6332Metric, symbol Device:R
- removed U1: MP1584EN_12V, Package_TO_SOT_SMD:SOT-23-8, symbol Driver:MP1584EN
- removed U2: MP1584EN_6V5, Package_TO_SOT_SMD:SOT-23-8, symbol Driver:MP1584EN
- removed U3: MP1584EN_5V, Package_TO_SOT_SMD:SOT-23-8, symbol Driver:MP1584EN
- removed U4, U5: DRV8876, Package_SO:WSON-8-1EP_2x2mm_P0.5mm_EP0.9x1.6mm, symbol Driver:DRV8876
- removed U6: TB6612FNG, Package_SO:SSOP-24_3.9x8.7mm_P0.635mm, symbol Driver:TB6612FNG
- removed U7: INA219, Package_TO_SOT_SMD:SOT-23-8, symbol Driver:INA219
- removed U8: PCF8574, Package_SO:SOIC-16_3.9x9.9mm_P1.27mm, symbol Driver:PCF8574
- added C17, C18, C19, C20, C21: 22uF, Capacitor_SMD:C_0805_2012Metric, symbol Device:C
- added C22, C23, C24, C25, C27, C28: 100nF, Capacitor_SMD:C_0402_1005Metric, symbol Device:C
- added C26: 10uF, Capacitor_SMD:C_0805_2012Metric, symbol Device:C
- added D1: SS54, Diode_SMD:D_SMA, symbol Diode:1N4148WS
- added D10, D11, D12, D13, D14, D15, D16, D6, D7, D8, D9: SS14, Diode_SMD:D_SOD-123, symbol Diode:1N4148WS
- added D17, D18, D19: SS34, Diode_SMD:D_SMA, symbol Diode:1N4148WS
- added D2: SMBJ24A, Diode_SMD:D_SMA, symbol Diode:1N4148WS
- added D20, D3: SMBJ12A, Diode_SMD:D_SMA, symbol Diode:1N4148WS
- added D4: SMBJ6V5, Diode_SMD:D_SMA, symbol Diode:1N4148WS
- added F1: 5A_PTC, Resistor_SMD:R_1206_3216Metric, symbol Device:R
- added F2: 1.5A, Resistor_SMD:R_1206_3216Metric, symbol Device:R
- added F3: 3A, Resistor_SMD:R_1206_3216Metric, symbol Device:R
- added F5: 3A_PTC, Resistor_SMD:R_1206_3216Metric, symbol Device:R
- added J1: J_24V_IN, Connector_JST:JST_XH_B2B-XH-A_1x02_P2.50mm_Vertical, symbol Connector_Generic:Conn_01x02
- added J10: J_STACK, Connector_PinHeader_2.54mm:PinHeader_2x20_P2.54mm_Vertical, symbol Connector_Generic:Conn_02x20_Odd_Even
- added J2: J_12V_UPS, Connector_JST:JST_XH_B2B-XH-A_1x02_P2.50mm_Vertical, symbol Connector_Generic:Conn_01x02
- added J3: J_BLDC, Connector_JST:JST_XH_B6B-XH-A_1x06_P2.50mm_Vertical, symbol Connector_Generic:Conn_01x06
- added J4: J_FAN, Connector_JST:JST_XH_B4B-XH-A_1x04_P2.50mm_Vertical, symbol Connector_Generic:Conn_01x04
- added J5: J_CID, Connector_JST:JST_XH_B4B-XH-A_1x04_P2.50mm_Vertical, symbol Connector_Generic:Conn_01x04
- added J6: J_CAN, Connector_JST:JST_XH_B4B-XH-A_1x04_P2.50mm_Vertical, symbol Connector_Generic:Conn_01x04
- added J7: J_BUZZER, Connector_JST:JST_PH_B2B-PH-K_1x02_P2.00mm_Vertical, symbol Connector_Generic:Conn_01x02
- added J8: J_SLD, Connector_JST:JST_XH_B12B-XH-A_1x12_P2.50mm_Vertical, symbol Connector_Generic:Conn_01x12
- added J9: J_PASD, Connector_JST:JST_XH_B16B-XH-A_1x16_P2.50mm_Vertical, symbol Connector_Generic:Conn_01x16
- added L1: 33uH, Inductor_SMD:L_1210_3225Metric, symbol Device:R
- added L2: 22uH, Inductor_SMD:L_1210_3225Metric, symbol Device:R
- added L4: 10uH, Inductor_SMD:L_1210_3225Metric, symbol Device:R
- added Q1, Q10, Q11, Q2, Q3, Q4, Q5, Q6, Q7, Q8, Q9: IRLML6344, Package_TO_SOT_SMD:SOT-23, symbol Transistor_FET:2N7002
- added R20: 10mR, Resistor_SMD:R_2512_6332Metric, symbol Device:R
- added R21: 100k, Resistor_SMD:R_0402_1005Metric, symbol Device:R
- added R22, R24, R26, R28, RPD1, RPD10, RPD11, RPD12, RPD2, RPD3, RPD4, RPD5, RPD6, RPD7, RPD8, RPD9: 10k, Resistor_SMD:R_0402_1005Metric, symbol Device:R
- added R23: 140k, Resistor_SMD:R_0402_1005Metric, symbol Device:R
- added R25: 71.5k, Resistor_SMD:R_0402_1005Metric, symbol Device:R
- added R27: 52.3k, Resistor_SMD:R_0402_1005Metric, symbol Device:R
- added R29: 120, Resistor_SMD:R_0402_1005Metric, symbol Device:R
- added RG1, RG10, RG11, RG12, RG2, RG3, RG4, RG5, RG6, RG7, RG8, RG9: 100, Resistor_SMD:R_0402_1005Metric, symbol Device:R
- added U1, U2: MP1584EN, Package_SO:SOIC-8_3.9x4.9mm_P1.27mm, symbol Connector_Generic:Conn_01x08
- added U3: ISO1050, Package_SO:SOIC-8_3.9x4.9mm_P1.27mm, symbol Connector_Generic:Conn_01x08
- added U4, U5: DRV8876, Package_SO:VSSOP-8_3.0x3.0mm_P0.65mm, symbol Connector_Generic:Conn_01x08
- added U6: TB6612FNG, Package_SO:SSOP-24_5.3x8.2mm_P0.65mm, symbol Connector_Generic:Conn_01x12
- added U7: INA219, Package_SO:SOIC-8_3.9x4.9mm_P1.27mm, symbol Connector_Generic:Conn_01x08
- added U8: PCF8574, Package_SO:SOIC-16_3.9x9.9mm_P1.27mm, symbol Connector_Generic:Conn_01x16
- added U9: TPS54531, Package_SO:SOIC-8_3.9x4.9mm_P1.27mm, symbol Connector_Generic:Conn_01x08
Connections:
- net BUZZER_PWM: now also Q12.1 (G), J10.38 (Pin_38), RG12.1, RG12.2, RPD12.1
- net CID_LACT1_EN: now also J10.21 (Pin_21), U4.3 (Pin_3)
- net CID_LACT1_PH: now also J10.22 (Pin_22), U4.4 (Pin_4)
- net CID_LACT2_EN: now also J10.23 (Pin_23), U5.3 (Pin_3)
- net CID_LACT2_PH: now also J10.24 (Pin_24), U5.4 (Pin_4)
- net FAN1_PWM: now also J10.27 (Pin_27), Q3.1 (G), RG3.1, RG3.2, RPD3.1
- net FAN2_PWM: now also J10.28 (Pin_28), Q4.1 (G), RG4.1, RG4.2, RPD4.1
- net I2C1_SCL: now also J10.35 (Pin_35), U7.6 (Pin_6), U8.13 (Pin_13)
- net I2C1_SDA: now also J10.36 (Pin_36), U7.5 (Pin_5), U8.14 (Pin_14)
- net PASD_PUMP_PWM: now also J10.15 (Pin_15), Q5.1 (G), RG5.1, RG5.2, RPD5.1
- net SLD_PUMP1_DIR: now also J10.30 (Pin_30), U6.5 (Pin_5)
- net SLD_PUMP1_PWM: now also J10.29 (Pin_29), U6.4 (Pin_4)
- net SLD_PUMP2_DIR: now also J10.32 (Pin_32), U6.9 (Pin_9)
- net SLD_PUMP2_PWM: now also J10.31 (Pin_31), U6.8 (Pin_8)
- net GND: now reaches Q12.2 (S)
- net GND: now also C17.2, C18.2, C19.1, C19.2, C20.2, C21.2, C22.2, C23.2, C24.2, C25.2, C27.2, C28.2, D18.1 (K), D18.2 (A), D2.2 (A), D20.2 (A), D3.2 (A), D4.1 (K), D4.2 (A), F3.1, F3.2, J1.2 (Pin_2), J10.10 (Pin_10), J10.25 (Pin_25), J10.26 (Pin_26), J10.5 (Pin_5), J10.6 (Pin_6), J10.7 (Pin_7), J10.8 (Pin_8), J10.9 (Pin_9), J2.2 (Pin_2), J3.2 (Pin_2), J8.12 (Pin_12), J9.15 (Pin_15), J9.16 (Pin_16), L2.1, L2.2, Q1.2 (S), Q10.2 (S), Q11.2 (S), Q2.2 (S), Q3.2 (S), Q4.2 (S), Q5.2 (S), Q6.2 (S), Q7.2 (S), Q8.2 (S), Q9.2 (S), R22.2, R24.2, R25.1, R25.2, R26.1, R26.2, R28.2, RPD1.2, RPD10.2, RPD11.2, RPD12.2, RPD2.2, RPD3.2, RPD4.2, RPD5.2, RPD6.2, RPD7.2, RPD8.2, RPD9.2, U1.2 (Pin_2), U2.2 (Pin_2), U2.3 (Pin_3), U2.4 (Pin_4), U2.6 (Pin_6), U3.2 (Pin_2), U4.2 (Pin_2), U5.2 (Pin_2), U6.3 (Pin_3), U7.4 (Pin_4), U7.7 (Pin_7), U7.8 (Pin_8), U8.1 (Pin_1), U8.16 (Pin_16), U8.2 (Pin_2), U8.3 (Pin_3), U9.2 (Pin_2)
- net BUZZ_D: now reaches Q12.3 (D)
- net BUZZ_D: now also J7.2 (Pin_2)
- new net +24V: J10.1 (Pin_1), J10.2 (Pin_2), J10.3 (Pin_3), J10.4 (Pin_4)
- new net +3V3: C23.1, C25.1, J10.13 (Pin_13), J10.14 (Pin_14), J8.11 (Pin_11), U3.1 (Pin_1), U6.12 (Pin_12), U6.2 (Pin_2), U8.15 (Pin_15)
- new net +5V: C17.1, C18.1, C20.1, C21.1, C26.1, D1.1 (K), D1.2 (A), D17.1 (K), D17.2 (A), D2.1 (K), F1.1, F1.2, F2.1, J1.1 (Pin_1), J10.11 (Pin_11), J10.12 (Pin_12), J3.1 (Pin_1), J7.1 (Pin_1), L1.1, L1.2, L4.1, L4.2, R20.1, R20.2, R21.1, R23.1, R27.1, U1.1 (Pin_1), U1.3 (Pin_3), U1.4 (Pin_4), U1.5 (Pin_5), U2.1 (Pin_1), U2.5 (Pin_5), U3.5 (Pin_5), U7.1 (Pin_1), U7.2 (Pin_2), U7.3 (Pin_3), U9.3 (Pin_3), U9.4 (Pin_4)
- new net 12V_OUT: C24.1, C27.1, C28.1, D10.1 (K), D11.1 (K), D12.1 (K), D13.1 (K), D14.1 (K), D15.1 (K), D16.1 (K), D19.1 (K), D19.2 (A), D20.1 (K), D3.1 (K), D6.1 (K), D7.1 (K), D8.1 (K), D9.1 (K), F2.2, F5.1, F5.2, J2.1 (Pin_1), J4.1 (Pin_1), J4.3 (Pin_3), J8.5 (Pin_5), J8.7 (Pin_7), J9.1 (Pin_1), J9.11 (Pin_11), J9.13 (Pin_13), J9.3 (Pin_3), J9.5 (Pin_5), J9.7 (Pin_7), J9.9 (Pin_9), R23.2, R24.1, U1.6 (Pin_6), U4.1 (Pin_1), U5.1 (Pin_1), U6.1 (Pin_1), U9.1 (Pin_1), U9.5 (Pin_5)
- new net BLDC_DIR: J10.40 (Pin_40), J3.5 (Pin_5)
- new net BLDC_EN: J10.39 (Pin_39), J3.4 (Pin_4)
- new net BLDC_PWM: J10.37 (Pin_37), J3.3 (Pin_3)
- new net CAN_H: J6.1 (Pin_1), R29.1, U3.7 (Pin_7)
- new net CAN_L: J6.2 (Pin_2), R29.2, U3.8 (Pin_8)
- new net FAN1_D: D8.2 (A), J4.2 (Pin_2), Q3.3 (D)
- new net FAN2_D: D9.2 (A), J4.4 (Pin_4), Q4.3 (D)
- new net FB_5V: C22.1, J10.16 (Pin_16), J5.2 (Pin_2), R21.2, R22.1, R27.2, R28.1, U4.6 (Pin_6), U9.6 (Pin_6)
- new net FDCAN1_RX: J10.19 (Pin_19), U3.4 (Pin_4)
- new net FDCAN1_TX: J10.20 (Pin_20), U3.3 (Pin_3)
- new net GND_ISO: C26.2, J6.3 (Pin_3), U3.6 (Pin_6)
- new net HX711_DOUT: J10.18 (Pin_18), J8.10 (Pin_10)
- new net HX711_SCK: J10.17 (Pin_17), J8.9 (Pin_9)
- new net LACT1_O1: J5.1 (Pin_1), U4.5 (Pin_5)
- new net LACT2_O1: J5.3 (Pin_3), U5.5 (Pin_5)
- new net LACT2_O2: J5.4 (Pin_4), U5.6 (Pin_6)
- new net PASD_V1: Q6.1 (G), RG6.1, RG6.2, RPD6.1, U8.4 (Pin_4)
- new net PASD_V2: Q7.1 (G), RG7.1, RG7.2, RPD7.1, U8.5 (Pin_5)
- new net PASD_V3: Q8.1 (G), RG8.1, RG8.2, RPD8.1, U8.6 (Pin_6)
- new net PASD_V4: Q9.1 (G), RG9.1, RG9.2, RPD9.1, U8.7 (Pin_7)
- new net PASD_V5: Q10.1 (G), RG10.1, RG10.2, RPD10.1, U8.8 (Pin_8)
- new net PASD_V6: Q11.1 (G), RG11.1, RG11.2, RPD11.1, U8.9 (Pin_9)
- new net PSOL1_D: D11.2 (A), J9.2 (Pin_2), Q6.3 (D)
- new net PSOL2_D: D12.2 (A), J9.4 (Pin_4), Q7.3 (D)
- new net PSOL3_D: D13.2 (A), J9.6 (Pin_6), Q8.3 (D)
- new net PSOL4_D: D14.2 (A), J9.8 (Pin_8), Q9.3 (D)
- new net PSOL5_D: D15.2 (A), J9.10 (Pin_10), Q10.3 (D)
- new net PSOL6_D: D16.2 (A), J9.12 (Pin_12), Q11.3 (D)
- new net PUMP1_O1: J8.1 (Pin_1), U6.6 (Pin_6)
- new net PUMP1_O2: J8.2 (Pin_2), U6.7 (Pin_7)
- new net PUMP2_O1: J8.3 (Pin_3), U6.10 (Pin_10)
- new net PUMP2_O2: J8.4 (Pin_4), U6.11 (Pin_11)
- new net PUMP_D: D10.2 (A), J9.14 (Pin_14), Q5.3 (D)
- new net Q1_G: J10.33 (Pin_33), Q1.1 (G), RG1.1, RG1.2, RPD1.1
- new net Q2_G: J10.34 (Pin_34), Q2.1 (G), RG2.1, RG2.2, RPD2.1
- new net SOL1_D: D6.2 (A), J8.6 (Pin_6), Q1.3 (D)
- new net SOL2_D: D7.2 (A), J8.8 (Pin_8), Q2.3 (D)
- no-connect marks 0 -> 15
Other:
- note added: "24V Input / Fuse / Protection"
- note added: "BLDC Motor Driver — DRV8876"
- note added: "Buck Converter 1 — MP1584EN (5V)"
- note added: "Buck Converter 2 — MP1584EN (6V5)"
- note added: "Buck Converter 3 — TPS54531 (12V)"
- note added: "CAN Transceiver — ISO1050"
- note added: "CID Motor Driver — DRV8876"
- note added: "Connectors — J_BUZZER, J_SLD, J_PASD"
- note added: "Connectors — J_FAN, J_CID, J_CAN"
- note added: "Current Sense — INA219"
- note added: "Dual H-Bridge — TB6612FNG"
- note added: "Fan Drivers (Q3-Q4)"
- note added: "I2C Expander — PCF8574"
- note added: "J_STACK — Board-to-Board 2x20"
- note added: "Pump / Buzzer Driver (Q5, Q12)"
- note added: "Solenoid Drivers (Q1-Q2)"
- note added: "Valve Drivers (Q6-Q11)"
- company: Epicura -> Epicura / Designed by Cyber_Lord
- title: Epicura Driver PCB -> Epicura Driver Board
